File: power.kicad_sch (KiCad schematic)
At the start: 24 parts, among them J6 USB 2.0 right angle, J8 POWER_MEASUREMENT, Q2 AO3401A, U2 USBLC6-2SC6, U3 TP4056, U4 ME6216 3V0

Commit message: WIP
Parts:
- J8, JP1: now left out of the parts list
- TH1: footprint Capacitor_SMD:C_1206_3216Metric -> Resistor_THT:R_Axial_DIN0204_L3.6mm_D1.6mm_P5.08mm_Horizontal; LCSC (none) -> C267088

Commit message: Use single FPC connector for debug signals and downstream
Parts:
- U3: footprint local:ESOP-8 -> Package_SO:SOP-8-1EP_4.57x4.57mm_P1.27mm_EP4.57x4.45mm
Changed lines of the file:
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@@
       (effects (font (size 1.27 1.27)))
     )
-    (property "Footprint" "local:ESOP-8" (at 157.48 130.81 0)
+    (property "Footprint" "Package_SO:SOP-8-1EP_4.57x4.57mm_P1.27mm_EP4.57x4.45mm" (at 157.48 130.81 0)
       (effects (font (size 1.27 1.27)) hide)
     )

Commit message: Resistor calculations
Parts:
- R19: value ? -> 18k; footprint Resistor_SMD:R_0402_1005Metric -> Resistor_SMD:R_0603_1608Metric
- R20: value ? -> 5k1
- R21: value ? -> 100k
Changed lines of the file:
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@@
     (stroke (width 0) (type default))
+  )
+  (polyline (pts (xy 204.47 139.7) (xy 185.42 119.38))
+    (stroke (width 0) (type dot))
   )
   (wire (pts (xy 146.05 124.46) (xy 146.05 127))
@@
     (stroke (width 0) (type default))
   )
+  (polyline (pts (xy 160.02 139.7) (xy 172.72 125.73))
+    (stroke (width 0) (type dot))
+  )
   (wire (pts (xy 232.41 125.73) (xy 232.41 130.81))
     (stroke (width 0) (type default))
@@
   (wire (pts (xy 194.31 116.84) (xy 194.31 114.3))
     (stroke (width 0) (type default))
+  )
+  (text_box "Battery capacity is 330mAh.\nRecommanded charge current is 0.2C,\nwhich is 330mAh * 0.2 = 66 mAh.\nResistor on PROG = 1V*1200 / IBat = 18180 Ohm.\nNearest 0603 resistor among JLCPCB's basic parts is 18 kOhm,\nwhich gives 66.7 mA = 0.202C."
+    (at 109.22 139.7 0) (size 64.77 13.97)
+    (stroke (width 0) (type dot))
+    (fill (type none))
+    (effects (font (size 1.27 1.27)) (justify left top))
+  )
+  (text_box "Resistor divider values were found using\n\"TP4056 resistor calc.ipynb\" in the project directory."
+    (at 179.07 139.7 0) (size 54.61 6.35)
+    (stroke (width 0) (type dot))
+    (fill (type none))
+    (effects (font (size 1.27 1.27)) (justify left top))
   )
   (label "CC1" (at 54.61 68.58 0) (fields_autoplaced)
@@
       (effects (font (size 1.27 1.27)) (justify left))
     )
-    (property "Value" "?" (at 175.768 124.4021 0)
-      (effects (font (size 1.27 1.27)) (justify left))
-    )
-    (property "Footprint" "Resistor_SMD:R_0402_1005Metric" (at 172.212 123.19 90)
+    (property "Value" "18k" (at 175.768 124.4021 0)
+      (effects (font (size 1.27 1.27)) (justify left))
+    )
+    (property "Footprint" "Resistor_SMD:R_0603_1608Metric" (at 172.212 123.19 90)
       (effects (font (size 1.27 1.27)) hide)
     )
@@
       (effects (font (size 1.27 1.27)) (justify left))
     )
-    (property "Value" "?" (at 185.928 114.2421 0)
+    (property "Value" "5k1" (at 185.928 114.2421 0)
       (effects (font (size 1.27 1.27)) (justify left))
     )
@@
       (effects (font (size 1.27 1.27)) (justify left))
     )
-    (property "Value" "?" (at 185.928 125.6721 0)
-      (effects (font (size 1.27 1.27)) (justify left))
-    )
+    (property "Value" "100k" (at 185.928 125.6721 0)
+      (effects (font (size 1.27 1.27)) (justify left))
+    )

Commit message: switch to JLCPCB version of USBC connect fp
Parts:
- J6: footprint Connector_USB:USB_C_Receptacle_G-Switch_GT-USB-7010ASV -> local:USB-C-SMD_G-SWITCH_GT-USB-7010ASV
Changed lines of the file:
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@@
       (effects (font (size 1.27 1.27)))
     )
-    (property "Footprint" "Connector_USB:USB_C_Receptacle_G-Switch_GT-USB-7010ASV" (at 40.64 78.74 0)
+    (property "Footprint" "local:USB-C-SMD_G-SWITCH_GT-USB-7010ASV" (at 40.64 78.74 0)
       (effects (font (size 1.27 1.27)) hide)
     )
